File: First week/untitled.brd (EAGLE design)
At the start: 72.1 x 77.1 mm, 7 parts

Commit message: change
Parts:
- moved TTL2 2.54 mm to (12.7, 34.3)
- moved U$1 2.54 mm to (30.5, 43.2)
Routing:
- net 3.3V: track 113.3 -> 32.3 mm, vias 2 -> 0
- net GND: track 200.1 -> 169.0 mm, vias 2 -> 0
- net B: track 10.8 -> 13.5 mm
- net A: track 14.3 -> 17.1 mm
- net SCL: track 27.8 -> 26.8 mm
- net RX1: track 12.8 -> 11.7 mm
- net TX1: track 12.8 -> 11.7 mm
- net SDA: track 24.2 -> 23.2 mm
- net PWM: track 29.1 -> 30.1 mm, vias 0 -> 2
- net 5V: track 166.4 -> 167.0 mm
- net DIRECTION: track 32.4 -> 32.2 mm, vias 2 -> 0

Commit message: change
Parts:
- moved TTL2 11.4 mm to (7.62, 24.1), turned to 270 degrees
- moved U$2 11.4 mm to (47.0, 55.9)
- moved U$1 9.16 mm to (22.9, 38.1)
- moved CYTRON 9.16 mm to (40.6, 19.1)
- moved TTL1 8.52 mm to (40.6, 31.8), turned to 90 degrees
- moved ENCODER 8.03 mm to (40.6, 10.2)
- moved POWER_BASE 7.62 mm to (22.9, 7.62)
Connections:
- new net QWRGF3A: U$1.PB_1
- new net WAF: U$1.PB_0
- net DIRECTION: no longer U$1.PB_0
- net PWM: no longer U$1.PB_1
- net RX1: now also U$1.PA_10; no longer U$1.PA_9
- net RX3: now also U$1.PB_11; no longer U$1.PB_10
- net TX1: now also U$1.PA_9; no longer U$1.PA_10
- net TX3: now also U$1.PB_10; no longer U$1.PB_11
Routing:
- net GND: track 169.0 -> 104.4 mm, vias 0 -> 2
- net 5V: track 167.0 -> 142.5 mm, vias 2 -> 0
- net DIRECTION: track 32.2 -> 12.8 mm
- net PWM: track 30.1 -> 12.8 mm, vias 2 -> 0
- net A: track 17.1 -> 14.6 mm
- net B: track 13.5 -> 11.0 mm
- net TX3: track 10.2 -> 7.62 mm
- net RX3: track 10.2 -> 7.62 mm
- net 3.3V: track 32.3 -> 29.8 mm
- net SDA: track 23.2 -> 20.6 mm
- net SCL: track 26.8 -> 24.2 mm
- net TX1: track 11.7 -> 10.2 mm
- net RX1: track 11.7 -> 10.2 mm
Other:
- board size 72.1 x 77.1 mm -> 60.6 x 69.5 mm
