File: First week/untitled.sch (EAGLE design)
At the start: 7 parts

Commit message: change
Changed lines of the file:
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@@
 <pinref part="U$1" gate="G$1" pin="GND@2"/>
 <wire x1="35.56" y1="7.62" x2="30.48" y2="7.62" width="0.1524" layer="91"/>
-<label x="30.48" y="7.62" size="1.778" layer="95" rot="R180" xref="yes"/>
 </segment>
 <segment>
 <pinref part="U$1" gate="G$1" pin="GND@3"/>
 <wire x1="35.56" y1="2.54" x2="30.48" y2="2.54" width="0.1524" layer="91"/>
-<label x="30.48" y="2.54" size="1.778" layer="95" rot="R180" xref="yes"/>
 </segment>
 <segment>
@@
 <pinref part="U$1" gate="G$1" pin="3.3V@2"/>
 <wire x1="35.56" y1="12.7" x2="30.48" y2="12.7" width="0.1524" layer="91"/>
-<label x="30.48" y="12.7" size="1.4224" layer="95" rot="R180" xref="yes"/>
 </segment>
 </net>

Commit message: change
Connections:
- new net QWRGF3A: U$1.PB_1
- new net WAF: U$1.PB_0
- net DIRECTION: no longer U$1.PB_0
- net PWM: no longer U$1.PB_1
- net RX1: now also U$1.PA_10; no longer U$1.PA_9
- net RX3: now also U$1.PB_11; no longer U$1.PB_10
- net TX1: now also U$1.PA_9; no longer U$1.PA_10
- net TX3: now also U$1.PB_10; no longer U$1.PB_11
Changed lines of the file:
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@@
-</segment>
-<segment>
-<pinref part="U$1" gate="G$1" pin="PB_0"/>
-<wire x1="35.56" y1="38.1" x2="30.48" y2="38.1" width="0.1524" layer="91"/>
 </segment>
 <segment>
@@
 <wire x1="116.84" y1="-2.54" x2="111.76" y2="-2.54" width="0.1524" layer="91"/>
 <label x="111.76" y="-2.54" size="1.4224" layer="95" rot="R180" xref="yes"/>
-</segment>
-<segment>
-<pinref part="U$1" gate="G$1" pin="PB_1"/>
-<wire x1="35.56" y1="33.02" x2="30.48" y2="33.02" width="0.1524" layer="91"/>
 </segment>
 <segment>
@@
 </segment>
 <segment>
-<pinref part="U$1" gate="G$1" pin="PB_11"/>
-<wire x1="35.56" y1="22.86" x2="30.48" y2="22.86" width="0.1524" layer="91"/>
-<label x="30.48" y="22.86" size="1.4224" layer="95" rot="R180" xref="yes"/>
+<pinref part="U$1" gate="G$1" pin="PB_10"/>
+<wire x1="35.56" y1="27.94" x2="30.48" y2="27.94" width="0.1524" layer="91"/>
+<label x="30.48" y="27.94" size="1.4224" layer="95" rot="R180" xref="yes"/>
 </segment>
 </net>
@@
 </segment>
 <segment>
-<pinref part="U$1" gate="G$1" pin="PB_10"/>
-<wire x1="35.56" y1="27.94" x2="30.48" y2="27.94" width="0.1524" layer="91"/>
-<label x="30.48" y="27.94" size="1.4224" layer="95" rot="R180" xref="yes"/>
+<pinref part="U$1" gate="G$1" pin="PB_11"/>
+<wire x1="35.56" y1="22.86" x2="30.48" y2="22.86" width="0.1524" layer="91"/>
+<label x="30.48" y="22.86" size="1.4224" layer="95" rot="R180" xref="yes"/>
 </segment>
 </net>
@@
 </segment>
 <segment>
-<pinref part="U$1" gate="G$1" pin="PA_10"/>
-<wire x1="76.2" y1="33.02" x2="81.28" y2="33.02" width="0.1524" layer="91"/>
-<label x="81.28" y="33.02" size="1.4224" layer="95" xref="yes"/>
+<pinref part="U$1" gate="G$1" pin="PA_9"/>
+<wire x1="76.2" y1="27.94" x2="81.28" y2="27.94" width="0.1524" layer="91"/>
+<label x="81.28" y="27.94" size="1.4224" layer="95" xref="yes"/>
 </segment>
 </net>
@@
 </segment>
 <segment>
-<pinref part="U$1" gate="G$1" pin="PA_9"/>
-<wire x1="76.2" y1="27.94" x2="81.28" y2="27.94" width="0.1524" layer="91"/>
-<label x="81.28" y="27.94" size="1.4224" layer="95" xref="yes"/>
+<pinref part="U$1" gate="G$1" pin="PA_10"/>
+<wire x1="76.2" y1="33.02" x2="81.28" y2="33.02" width="0.1524" layer="91"/>
+<label x="81.28" y="33.02" size="1.4224" layer="95" xref="yes"/>
 </segment>
 </net>
+<net name="WAF" class="0">
+<segment>
+<pinref part="U$1" gate="G$1" pin="PB_0"/>
+<wire x1="35.56" y1="38.1" x2="30.48" y2="38.1" width="0.1524" layer="91"/>
+</segment>
+</net>
+<net name="QWRGF3A" class="0">
+<segment>
+<pinref part="U$1" gate="G$1" pin="PB_1"/>
+<wire x1="35.56" y1="33.02" x2="30.48" y2="33.02" width="0.1524" layer="91"/>
+</segment>
+</net>
